Commit message: feat(model): 按《天工行者Dex V3 关键参数表》统一模型参数
- urdf/tiangong3.urdf 与 .xacro：39 个 link 的质量/质心/惯量、31 个 revolute 关节的下限/上限/力矩/速度对齐 CSV

- 两份模型文件自此除根标签外完全一致（原 20 个关节限位差异已消除）

- 模型总质量 63.272 -> 65.818 kg

- 新增 关键参数/URDF关键参数表 - 天工行者Dex(V3).csv 并加入 CMakeLists install

- 同步 scripts/validate.py、docs/model.md、docs/joints.md、CHANGELOG.md

File: src/tiangong3_urdf/urdf/tiangong3.urdf (robot description, URDF)
Before this commit: robot tiangong3_urdf, 39 links, 38 joints
Links:
- link ankle_pitch_l_link: mass 0.142658 -> 0.122342
- link ankle_pitch_r_link: mass 0.142658 -> 0.122342
- link ankle_roll_l_link: mass 0.888892 -> 0.826437
- link ankle_roll_r_link: mass 0.888892 -> 0.826437
- link elbow_pitch_l_link: mass 0.647211 -> 0.762706
- link elbow_pitch_r_link: mass 0.647211 -> 0.762706
- link elbow_yaw_l_link: mass 0.229689 -> 0.31993
- link elbow_yaw_r_link: mass 0.229689 -> 0.31993
- link head_pitch_link: mass 0.067829 -> 0.077424
- link head_yaw_link: mass 0.95297 -> 1.057204
- link hip_pitch_l_link: mass 2.221379 -> 2.427595
- link hip_pitch_r_link: mass 2.221379 -> 2.427595
- link hip_roll_l_link: mass 0.560034 -> 0.578439
- link hip_roll_r_link: mass 0.560034 -> 0.578439
- link hip_yaw_l_link: mass 5.658158 -> 5.766953
- link hip_yaw_r_link: mass 5.658158 -> 5.766953
- link knee_pitch_l_link: mass 3.158584 -> 3.14544
- link knee_pitch_r_link: mass 3.158584 -> 3.14544
- link left_tcp_link: mass 0.457436 -> 0.384094
- link pelvis: mass 10.579253 -> 11.09264
- link right_tcp_link: mass 0.457436 -> 0.384094
- link shoulder_pitch_l_link: mass 0.914808 -> 0.967698
- link shoulder_pitch_r_link: mass 0.914808 -> 0.967698
- link shoulder_roll_l_link: mass 0.319153 -> 0.460858
- link shoulder_roll_r_link: mass 0.319153 -> 0.460858
- link shoulder_yaw_l_link: mass 1.502215 -> 1.53899
- link shoulder_yaw_r_link: mass 1.502215 -> 1.53899
- link waist_pitch_link: mass 10.403447 -> 9.973084
- link waist_roll_link: mass 3.595194 -> 3.894484
- link waist_yaw_link: mass 1.688374 -> 2.135803
- link wrist_pitch_l_link: mass 0.931823 -> 1.089228
- link wrist_pitch_r_link: mass 0.931823 -> 1.089228
- link wrist_roll_l_link: mass 0.12 -> 0.162372
- link wrist_roll_r_link: mass 0.12 -> 0.162372
Joints:
- joint ankle_pitch_l_joint: limit lower=-1.2217304763960306 upper=0.5235987755982988 effort=55.0 velocity=14.137166941154069 -> lower=-1.1868238913561442 upper=0.5235987755982988 effort=55.0 velocity=14.137166941154069
- joint ankle_pitch_r_joint: limit lower=-1.2217304763960306 upper=0.5235987755982988 effort=55.0 velocity=14.137166941154069 -> lower=-1.1868238913561442 upper=0.5235987755982988 effort=55.0 velocity=14.137166941154069
- joint elbow_yaw_l_joint: limit lower=-2.844886680750757 upper=2.844886680750757 effort=25.0 velocity=12.217653829810706 -> lower=-2.844886680750757 upper=2.844886680750757 effort=40.0 velocity=18.325957145940457
- joint elbow_yaw_r_joint: limit lower=-2.844886680750757 upper=2.844886680750757 effort=25.0 velocity=12.217653829810706 -> lower=-2.844886680750757 upper=2.844886680750757 effort=40.0 velocity=18.325957145940457
- joint waist_pitch_joint: limit lower=-0.5235987755982988 upper=0.9599310885968813 effort=150.0 velocity=13.82300767579509 -> lower=-0.5235987755982988 upper=0.8726646259971648 effort=150.0 velocity=13.82300767579509
- joint waist_yaw_joint: limit lower=-2.6179938779914944 upper=3.2288591161895095 effort=91.0 velocity=9.42477796076938 -> lower=-2.6179938779914944 upper=3.2288591161895095 effort=200.0 velocity=10.053096491487338
- joint wrist_pitch_l_joint: limit lower=-1.3264502315156903 upper=1.3264502315156903 effort=25.0 velocity=12.217653829810706 -> lower=-1.3264502315156903 upper=1.3264502315156903 effort=40.0 velocity=18.325957145940457
- joint wrist_pitch_r_joint: limit lower=-1.3264502315156903 upper=1.3264502315156903 effort=25.0 velocity=12.217653829810706 -> lower=-1.3264502315156903 upper=1.3264502315156903 effort=40.0 velocity=18.325957145940457
- joint wrist_roll_l_joint: limit lower=-1.3264502315156903 upper=1.3264502315156903 effort=25.0 velocity=12.217653829810706 -> lower=-1.3264502315156903 upper=1.3264502315156903 effort=40.0 velocity=18.325957145940457
- joint wrist_roll_r_joint: limit lower=-1.3264502315156903 upper=1.3264502315156903 effort=25.0 velocity=12.217653829810706 -> lower=-1.3264502315156903 upper=1.3264502315156903 effort=40.0 velocity=18.325957145940457
