Commit message: feat(model): 按《天工行者Dex V3 关键参数表》统一模型参数
- urdf/tiangong3.urdf 与 .xacro：39 个 link 的质量/质心/惯量、31 个 revolute 关节的下限/上限/力矩/速度对齐 CSV

- 两份模型文件自此除根标签外完全一致（原 20 个关节限位差异已消除）

- 模型总质量 63.272 -> 65.818 kg

- 新增 关键参数/URDF关键参数表 - 天工行者Dex(V3).csv 并加入 CMakeLists install

- 同步 scripts/validate.py、docs/model.md、docs/joints.md、CHANGELOG.md

File: src/tiangong3_urdf/urdf/tiangong3.urdf.xacro (robot description, xacro)
@@ -3,7 +3,7 @@
   <link name="pelvis">
     <inertial>
-      <origin xyz="0.000772 -0.000475 -0.060309" rpy="0 0 0" />
-      <mass value="10.579253" />
-      <inertia ixx="0.089056" ixy="-2.6e-05" ixz="-0.00093" iyy="0.072375" iyz="0.000499" izz="0.069877" />
+      <origin xyz="0.000058 0.000357 -0.054446" rpy="0 0 0" />
+      <mass value="11.09264" />
+      <inertia ixx="0.07166" ixy="-0.000356" ixz="-0.002017" iyy="0.065195" iyz="0.000097" izz="0.049883" />
     </inertial>
     <visual>
@@ -25,7 +25,7 @@
   <link name="hip_pitch_l_link">
     <inertial>
-      <origin xyz="0.009589 0.069327 -0.024358" rpy="0 0 0" />
-      <mass value="2.221379" />
-      <inertia ixx="0.004839" ixy="-0.00014" ixz="8.3e-05" iyy="0.003411" iyz="0.000185" izz="0.003611" />
+      <origin xyz="0.009137 0.070235 -0.024662" rpy="0 0 0" />
+      <mass value="2.427595" />
+      <inertia ixx="0.00525" ixy="-0.000103" ixz="0.000064" iyy="0.003734" iyz="0.000156" izz="0.003966" />
     </inertial>
     <visual>
@@ -50,11 +50,11 @@
     <child link="hip_pitch_l_link" />
     <axis xyz="0 1 0" />
-    <limit lower="-3.141592653589793" upper="2.8797932657906435" effort="235.0" velocity="16.755160819145562" />
+    <limit lower="-3.0543261909900763" upper="2.792526803190927" effort="235.0" velocity="16.755160819145562" />
   </joint>
   <link name="hip_roll_l_link">
     <inertial>
-      <origin xyz="-0.000767 -4.3e-05 -0.03918" rpy="0 0 0" />
-      <mass value="0.560034" />
-      <inertia ixx="0.0011" ixy="1e-06" ixz="3.2e-05" iyy="0.001743" iyz="0.0" izz="0.001475" />
+      <origin xyz="-0.002953 -0.000095 -0.037153" rpy="0 0 0" />
+      <mass value="0.578439" />
+      <inertia ixx="0.001108" ixy="0.000003" ixz="0.00004" iyy="0.001818" iyz="-0.000001" izz="0.001505" />
     </inertial>
     <visual>
@@ -83,7 +83,7 @@
   <link name="hip_yaw_l_link">
     <inertial>
-      <origin xyz="0.001014 -0.022912 -0.125892" rpy="0 0 0" />
-      <mass value="5.658158" />
-      <inertia ixx="0.045606" ixy="-0.000415" ixz="-0.000509" iyy="0.042833" iyz="-0.00159" izz="0.01441" />
+      <origin xyz="0.001274 -0.023741 -0.132464" rpy="0 0 0" />
+      <mass value="5.766953" />
+      <inertia ixx="0.047987" ixy="-0.000286" ixz="-0.000443" iyy="0.0454" iyz="-0.00214" izz="0.015312" />
     </inertial>
     <visual>
@@ -108,11 +108,11 @@
     <child link="hip_yaw_l_link" />
     <axis xyz="0 0 1" />
-    <limit lower="-1.3962634015954636" upper="4.537856055185257" effort="150.0" velocity="13.82300767579509" />
+    <limit lower="-1.3962634015954636" upper="4.4505895925855405" effort="150.0" velocity="13.82300767579509" />
   </joint>
   <link name="knee_pitch_l_link">
     <inertial>
-      <origin xyz="0.02218 -0.000444 -0.151985" rpy="0 0 0" />
-      <mass value="3.158584" />
-      <inertia ixx="0.03449" ixy="-9.9e-05" ixz="-0.002541" iyy="0.034832" iyz="-0.000815" izz="0.004008" />
+      <origin xyz="0.024736 0.000774 -0.150638" rpy="0 0 0" />
+      <mass value="3.14544" />
+      <inertia ixx="0.032343" ixy="-0.000047" ixz="-0.001178" iyy="0.032448" iyz="-0.000677" izz="0.003699" />
     </inertial>
     <visual>
@@ -141,7 +141,7 @@
   <link name="ankle_pitch_l_link">
     <inertial>
-      <origin xyz="0.0 0.0 0.0" rpy="0 0 0" />
-      <mass value="0.142658" />
-      <inertia ixx="2.3e-05" ixy="0.0" ixz="0.0" iyy="3.2e-05" iyz="0.0" izz="4.9e-05" />
+      <origin xyz="0 0 0" rpy="0 0 0" />
+      <mass value="0.122342" />
+      <inertia ixx="0.000038" ixy="0" ixz="0" iyy="0.000025" iyz="0" izz="0.000018" />
     </inertial>
     <visual>
@@ -166,11 +166,11 @@
     <child link="ankle_pitch_l_link" />
     <axis xyz="0 1 0" />
-    <limit lower="-1.2217304763960306" upper="0.5235987755982988" effort="55.0" velocity="14.137166941154069" />
+    <limit lower="-1.1868238913561442" upper="0.5235987755982988" effort="55.0" velocity="14.137166941154069" />
   </joint>
   <link name="ankle_roll_l_link">
     <inertial>
-      <origin xyz="0.024536 -1.7e-05 -0.033593" rpy="0 0 0" />
-      <mass value="0.888892" />
-      <inertia ixx="0.000779" ixy="-1e-06" ixz="0.000255" iyy="0.004839" iyz="1e-06" izz="0.005126" />
+      <origin xyz="0.025067 0.000002 -0.033303" rpy="0 0 0" />
+      <mass value="0.826437" />
+      <inertia ixx="0.000702" ixy="0" ixz="0.000201" iyy="0.004499" iyz="0" izz="0.00479" />
     </inertial>
     <visual>
@@ -199,7 +199,7 @@
   <link name="hip_pitch_r_link">
     <inertial>
-      <origin xyz="0.009589 -0.069327 -0.024358" rpy="0 0 0" />
-      <mass value="2.221379" />
-      <inertia ixx="0.004839" ixy="0.00014" ixz="8.3e-05" iyy="0.003411" iyz="-0.000185" izz="0.003611" />
+      <origin xyz="0.009137 -0.070235 -0.024662" rpy="0 0 0" />
+      <mass value="2.427595" />
+      <inertia ixx="0.00525" ixy="0.000103" ixz="0.000064" iyy="0.003734" iyz="-0.000156" izz="0.003966" />
     </inertial>
     <visual>
@@ -224,11 +224,11 @@
     <child link="hip_pitch_r_link" />
     <axis xyz="0 1 0" />
-    <limit lower="-3.141592653589793" upper="2.8797932657906435" effort="235.0" velocity="16.755160819145562" />
+    <limit lower="-3.0543261909900763" upper="2.792526803190927" effort="235.0" velocity="16.755160819145562" />
   </joint>
   <link name="hip_roll_r_link">
     <inertial>
-      <origin xyz="-0.000767 4.3e-05 -0.03918" rpy="0 0 0" />
-      <mass value="0.560034" />
-      <inertia ixx="0.0011" ixy="-1e-06" ixz="3.2e-05" iyy="0.001743" iyz="0.0" izz="0.001475" />
+      <origin xyz="-0.002953 0.000095 -0.037153" rpy="0 0 0" />
+      <mass value="0.578439" />
+      <inertia ixx="0.001108" ixy="-0.000003" ixz="0.00004" iyy="0.001818" iyz="0.000001" izz="0.001505" />
     </inertial>
     <visual>
@@ -257,7 +257,7 @@
   <link name="hip_yaw_r_link">
     <inertial>
-      <origin xyz="0.001014 0.022912 -0.125892" rpy="0 0 0" />
-      <mass value="5.658158" />
-      <inertia ixx="0.045606" ixy="0.000415" ixz="-0.000509" iyy="0.042833" iyz="0.00159" izz="0.01441" />
+      <origin xyz="0.001274 0.023741 -0.132464" rpy="0 0 0" />
+      <mass value="5.766953" />
+      <inertia ixx="0.047987" ixy="0.000286" ixz="-0.000443" iyy="0.0454" iyz="0.00214" izz="0.015312" />
     </inertial>
     <visual>
@@ -282,11 +282,11 @@
     <child link="hip_yaw_r_link" />
     <axis xyz="0 0 1" />
-    <limit lower="-4.537856055185257" upper="1.3962634015954636" effort="150.0" velocity="13.82300767579509" />
+    <limit lower="-4.4505895925855405" upper="1.3962634015954636" effort="150.0" velocity="13.82300767579509" />
   </joint>
   <link name="knee_pitch_r_link">
     <inertial>
-      <origin xyz="0.02218 0.000444 -0.151985" rpy="0 0 0" />
-      <mass value="3.158584" />
-      <inertia ixx="0.03449" ixy="9.9e-05" ixz="-0.002541" iyy="0.034832" iyz="0.000815" izz="0.004008" />
+      <origin xyz="0.024736 -0.000774 -0.150638" rpy="0 0 0" />
+      <mass value="3.14544" />
+      <inertia ixx="0.032343" ixy="0.000047" ixz="-0.001178" iyy="0.032448" iyz="0.000677" izz="0.003699" />
     </inertial>
     <visual>
@@ -315,7 +315,7 @@
   <link name="ankle_pitch_r_link">
     <inertial>
-      <origin xyz="0.0 0.0 0.0" rpy="0 0 0" />
-      <mass value="0.142658" />
-      <inertia ixx="2.3e-05" ixy="0.0" ixz="0.0" iyy="3.2e-05" iyz="0.0" izz="4.9e-05" />
+      <origin xyz="0 0 0" rpy="0 0 0" />
+      <mass value="0.122342" />
+      <inertia ixx="0.000038" ixy="0" ixz="0" iyy="0.000025" iyz="0" izz="0.000018" />
     </inertial>
     <visual>
@@ -340,11 +340,11 @@
     <child link="ankle_pitch_r_link" />
     <axis xyz="0 1 0" />
-    <limit lower="-1.2217304763960306" upper="0.5235987755982988" effort="55.0" velocity="14.137166941154069" />
+    <limit lower="-1.1868238913561442" upper="0.5235987755982988" effort="55.0" velocity="14.137166941154069" />
   </joint>
   <link name="ankle_roll_r_link">
     <inertial>
-      <origin xyz="0.024536 1.7e-05 -0.033593" rpy="0 0 0" />
-      <mass value="0.888892" />
-      <inertia ixx="0.000779" ixy="1e-06" ixz="0.000255" iyy="0.004839" iyz="-1e-06" izz="0.005126" />
+      <origin xyz="0.025067 -0.000002 -0.033303" rpy="0 0 0" />
+      <mass value="0.826437" />
+      <inertia ixx="0.000702" ixy="0" ixz="0.000201" iyy="0.004499" iyz="0" izz="0.00479" />
     </inertial>
     <visual>
@@ -373,7 +373,7 @@
   <link name="waist_yaw_link">
     <inertial>
-      <origin xyz="-0.001947 -0.000934 0.044217" rpy="0 0 0" />
-      <mass value="1.688374" />
-      <inertia ixx="0.002227" ixy="-4.1e-05" ixz="0.000158" iyy="0.002467" iyz="4.1e-05" izz="0.001927" />
+      <origin xyz="-0.001865 -0.000919 0.038314" rpy="0 0 0" />
+      <mass value="2.135803" />
+      <inertia ixx="0.00317" ixy="-0.000064" ixz="0.000201" iyy="0.003374" iyz="0.000084" izz="0.00233" />
     </inertial>
     <visual>
@@ -398,11 +398,11 @@
     <child link="waist_yaw_link" />
     <axis xyz="0 0 1" />
-    <limit lower="-2.740166925631097" upper="3.2288591161895095" effort="91.0" velocity="9.42477796076938" />
+    <limit lower="-2.6179938779914944" upper="3.2288591161895095" effort="200.0" velocity="10.053096491487338" />
   </joint>
   <link name="waist_roll_link">
     <inertial>
-      <origin xyz="-0.006103 -0.006401 0.0721" rpy="0 0 0" />
-      <mass value="3.595194" />
-      <inertia ixx="0.014592" ixy="0.000884" ixz="0.000209" iyy="0.007122" iyz="0.00011" izz="0.014704" />
+      <origin xyz="-0.007689 -0.005293 0.069696" rpy="0 0 0" />
+      <mass value="3.894484" />
+      <inertia ixx="0.015903" ixy="0.000774" ixz="0.000017" iyy="0.008878" iyz="0.000087" izz="0.016296" />
     </inertial>
     <visual>
@@ -431,7 +431,7 @@
   <link name="waist_pitch_link">
     <inertial>
-      <origin xyz="-0.002698 0.001618 0.182841" rpy="0 0 0" />
-      <mass value="10.403447" />
-      <inertia ixx="0.164891" ixy="-0.000251" ixz="0.002448" iyy="0.134319" iyz="-0.000324" izz="0.093659" />
+      <origin xyz="-0.004236 0.001466 0.18249" rpy="0 0 0" />
+      <mass value="9.973084" />
+      <inertia ixx="0.157779" ixy="-0.000188" ixz="0.002657" iyy="0.120648" iyz="0.000217" izz="0.094423" />
     </inertial>
     <visual>
@@ -456,11 +456,11 @@
     <child link="waist_pitch_link" />
     <axis xyz="0 1 0" />
-    <limit lower="-0.5235987755982988" upper="0.9599310885968813" effort="150.0" velocity="13.82300767579509" />
+    <limit lower="-0.5235987755982988" upper="0.8726646259971648" effort="150.0" velocity="13.82300767579509" />
   </joint>
   <link name="head_yaw_link">
     <inertial>
-      <origin xyz="0.015357 0.000986 0.023702" rpy="0 0 0" />
-      <mass value="0.95297" />
-      <inertia ixx="0.001542" ixy="-1.5e-05" ixz="-9.7e-05" iyy="0.001564" iyz="-1e-06" izz="0.002195" />
+      <origin xyz="0.013079 -0.000325 0.024349" rpy="0 0 0" />
+      <mass value="1.057204" />
+      <inertia ixx="0.002048" ixy="0.00006" ixz="-0.000057" iyy="0.001827" iyz="0.00005" izz="0.002642" />
     </inertial>
     <visual>
@@ -489,7 +489,7 @@
   <link name="head_pitch_link">
     <inertial>
-      <origin xyz="-0.001681 0.0042 -0.00014" rpy="0 0 0" />
-      <mass value="0.067829" />
-      <inertia ixx="7.1e-05" ixy="3e-06" ixz="0.0" iyy="2.2e-05" iyz="0.0" izz="6.5e-05" />
+      <origin xyz="-0.002436 0.002451 -0.000046" rpy="0 0 0" />
+      <mass value="0.077424" />
+      <inertia ixx="0.000092" ixy="0.000002" ixz="0" iyy="0.000024" iyz="0" izz="0.000086" />
     </inertial>
     <visual>
@@ -514,5 +514,5 @@
     <child link="head_pitch_link" />
     <axis xyz="0 1 0" />
-    <limit lower="-0.9599310885968813" upper="0.2617993877991494" effort="6.3" velocity="7.644542123735163" />
+    <limit lower="-0.8726646259971648" upper="0.2617993877991494" effort="6.3" velocity="7.644542123735163" />
   </joint>
   <link name="camera_head_link">
@@ -520,5 +520,5 @@
       <origin xyz="0.010986 -0.000307 -0.016475" rpy="0 0 0" />
       <mass value="0.1" />
-      <inertia ixx="1.6e-05" ixy="0.0" ixz="0.0" iyy="8e-05" iyz="0.0" izz="7.7e-05" />
+      <inertia ixx="0.000016" ixy="0" ixz="0" iyy="0.00008" iyz="0" izz="0.000077" />
     </inertial>
     <visual>
@@ -546,7 +546,7 @@
   <link name="radar_head_link">
     <inertial>
-      <origin xyz="-0.0002 -6e-06 -0.017365" rpy="0 0 0" />
+      <origin xyz="-0.0002 -0.000006 -0.017365" rpy="0 0 0" />
       <mass value="0.265" />
-      <inertia ixx="0.000124" ixy="0.0" ixz="0.0" iyy="0.000133" iyz="0.0" izz="0.000132" />
+      <inertia ixx="0.000124" ixy="0" ixz="0" iyy="0.000133" iyz="0" izz="0.000132" />
     </inertial>
     <visual>
@@ -576,5 +576,5 @@
       <origin xyz="0.001734 0.001046 -0.009253" rpy="0 0 0" />
       <mass value="0.008" />
-      <inertia ixx="1e-06" ixy="0.0" ixz="0.0" iyy="1e-06" iyz="0.0" izz="1e-06" />
+      <inertia ixx="0.000001" ixy="0" ixz="0" iyy="0.000001" iyz="0" izz="0.000001" />
     </inertial>
     <visual>
@@ -602,7 +602,7 @@
   <link name="shoulder_pitch_l_link">
     <inertial>
-      <origin xyz="0.006861 0.060647 -2.7e-05" rpy="0 0 0" />
-      <mass value="0.914808" />
-      <inertia ixx="0.000763" ixy="-4.9e-05" ixz="-1e-06" iyy="0.000912" iyz="0.0" izz="0.001164" />
+      <origin xyz="0.004116 0.061287 -0.000026" rpy="0 0 0" />
+      <mass value="0.967698" />
+      <inertia ixx="0.000726" ixy="-0.000031" ixz="-0.000001" iyy="0.001028" iyz="0" izz="0.00128" />
     </inertial>
     <visual>
@@ -627,11 +627,11 @@
     <child link="shoulder_pitch_l_link" />
     <axis xyz="0 1 0" />
-    <limit lower="-2.9670597283903604" upper="2.9670597283903604" effort="90.0" velocity="7.218332720398149" />
+    <limit lower="-2.844886680750757" upper="2.844886680750757" effort="90.0" velocity="7.218332720398149" />
   </joint>
   <link name="shoulder_roll_l_link">
     <inertial>
-      <origin xyz="-0.000672 0.0 -0.043313" rpy="0 0 0" />
-      <mass value="0.319153" />
-      <inertia ixx="0.000764" ixy="0.0" ixz="-4e-06" iyy="0.000936" iyz="0.0" izz="0.000544" />
+      <origin xyz="0.000619 -0.000505 -0.048667" rpy="0 0 0" />
+      <mass value="0.460858" />
+      <inertia ixx="0.00085" ixy="-0.000001" ixz="-0.000033" iyy="0.00105" iyz="-0.000005" izz="0.000594" />
     </inertial>
     <visual>
@@ -656,11 +656,11 @@
     <child link="shoulder_roll_l_link" />
     <axis xyz="1 0 0" />
-    <limit lower="-0.2617993877991494" upper="3.4033920413889422" effort="90.0" velocity="7.218332720398149" />
+    <limit lower="-0.19198621771937624" upper="3.3335788713091694" effort="90.0" velocity="7.218332720398149" />
   </joint>
   <link name="shoulder_yaw_l_link">
     <inertial>
-      <origin xyz="0.009141 0.003692 -0.094058" rpy="0 0 0" />
-      <mass value="1.502215" />
-      <inertia ixx="0.007803" ixy="-6.8e-05" ixz="0.000939" iyy="0.007535" iyz="0.000395" izz="0.001334" />
+      <origin xyz="0.010088 0.004252 -0.094438" rpy="0 0 0" />
+      <mass value="1.53899" />
+      <inertia ixx="0.008548" ixy="-0.000047" ixz="0.000995" iyy="0.008121" iyz="0.000389" izz="0.001454" />
     </inertial>
     <visual>
@@ -685,11 +685,11 @@
     <child link="shoulder_yaw_l_link" />
     <axis xyz="0 0 1" />
-    <limit lower="-2.9670597283903604" upper="2.9670597283903604" effort="50.0" velocity="11.455294012539582" />
+    <limit lower="-2.844886680750757" upper="2.844886680750757" effort="50.0" velocity="11.455294012539582" />
   </joint>
   <link name="elbow_pitch_l_link">
     <inertial>
-      <origin xyz="-0.017311 0.000579 -0.066888" rpy="0 0 0" />
-      <mass value="0.647211" />
-      <inertia ixx="0.001355" ixy="-7e-06" ixz="-0.00011" iyy="0.001235" iyz="-2.4e-05" izz="0.000703" />
+      <origin xyz="-0.017074 0.00081 -0.061526" rpy="0 0 0" />
+      <mass value="0.762706" />
+      <inertia ixx="0.001489" ixy="-0.000006" ixz="-0.000113" iyy="0.001346" iyz="-0.000024" izz="0.000806" />
     </inertial>
     <visual>
@@ -714,11 +714,11 @@
     <child link="elbow_pitch_l_link" />
     <axis xyz="0 1 0" />
-    <limit lower="-2.6179938779914944" upper="0.2617993877991494" effort="50.0" velocity="11.455294012539582" />
+    <limit lower="-2.548180707911721" upper="0.19198621771937624" effort="50.0" velocity="11.455294012539582" />
   </joint>
   <link name="elbow_yaw_l_link">
     <inertial>
-      <origin xyz="0.001113 0.005481 -0.05106" rpy="0 0 0" />
-      <mass value="0.229689" />
-      <inertia ixx="0.000368" ixy="0.0" ixz="-1e-06" iyy="0.00029" iyz="-8e-06" izz="0.000206" />
+      <origin xyz="-0.000303 0.004743 -0.052097" rpy="0 0 0" />
+      <mass value="0.31993" />
+      <inertia ixx="0.000519" ixy="-0.000001" ixz="0.000001" iyy="0.000404" iyz="0.000017" izz="0.000291" />
     </inertial>
     <visual>
@@ -743,11 +743,11 @@
     <child link="elbow_yaw_l_link" />
     <axis xyz="0 0 1" />
-    <limit lower="-2.9670597283903604" upper="2.9670597283903604" effort="25.0" velocity="12.217653829810706" />
+    <limit lower="-2.844886680750757" upper="2.844886680750757" effort="40.0" velocity="18.325957145940457" />
   </joint>
   <link name="wrist_pitch_l_link">
     <inertial>
-      <origin xyz="0.000815 0.001368 -0.031332" rpy="0 0 0" />
-      <mass value="0.931823" />
-      <inertia ixx="0.00154" ixy="1e-06" ixz="2.6e-05" iyy="0.001556" iyz="-4e-05" izz="0.000638" />
+      <origin xyz="-0.000656 -0.000789 -0.02945" rpy="0 0 0" />
+      <mass value="1.089228" />
+      <inertia ixx="0.0018" ixy="-0.000001" ixz="-0.000025" iyy="0.001748" iyz="0.00003" izz="0.000788" />
     </inertial>
     <visual>
@@ -772,11 +772,11 @@
     <child link="wrist_pitch_l_link" />
     <axis xyz="0 1 0" />
-    <limit lower="-1.3962634015954636" upper="1.3962634015954636" effort="25.0" velocity="12.217653829810706" />
+    <limit lower="-1.3264502315156903" upper="1.3264502315156903" effort="40.0" velocity="18.325957145940457" />
   </joint>
   <link name="wrist_roll_l_link">
     <inertial>
-      <origin xyz="0.015458 0.0 -0.02345" rpy="0 0 0" />
-      <mass value="0.12" />
-      <inertia ixx="8.7e-05" ixy="0.0" ixz="-3.5e-05" iyy="0.000104" iyz="0.0" izz="7.5e-05" />
+      <origin xyz="0.015688 0.000009 -0.022145" rpy="0 0 0" />
+      <mass value="0.162372" />
+      <inertia ixx="0.000107" ixy="0" ixz="-0.000043" iyy="0.000127" iyz="0" izz="0.000098" />
     </inertial>
     <visual>
@@ -801,11 +801,11 @@
     <child link="wrist_roll_l_link" />
     <axis xyz="1 0 0" />
-    <limit lower="-1.3962634015954636" upper="1.3962634015954636" effort="25.0" velocity="12.217653829810706" />
+    <limit lower="-1.3264502315156903" upper="1.3264502315156903" effort="40.0" velocity="18.325957145940457" />
   </joint>
   <link name="left_tcp_link">
     <inertial>
-      <origin xyz="0.002425 -0.002564 -0.054678" rpy="0 0 0" />
-      <mass value="0.457436" />
-      <inertia ixx="0.000482" ixy="2.6e-05" ixz="-8e-06" iyy="0.000603" iyz="-3.2e-05" izz="0.000441" />
+      <origin xyz="0.003693 -0.005984 -0.055343" rpy="0 0 0" />
+      <mass value="0.384094" />
+      <inertia ixx="0.000428" ixy="0.000016" ixz="-0.000006" iyy="0.000543" iyz="-0.000042" izz="0.000378" />
     </inertial>
     <visual>
@@ -833,7 +833,7 @@
   <link name="shoulder_pitch_r_link">
     <inertial>
-      <origin xyz="0.006861 -0.060647 -2.7e-05" rpy="0 0 0" />
-      <mass value="0.914808" />
-      <inertia ixx="0.000763" ixy="4.9e-05" ixz="-1e-06" iyy="0.000912" iyz="0.0" izz="0.001164" />
+      <origin xyz="0.004116 -0.061287 -0.000026" rpy="0 0 0" />
+      <mass value="0.967698" />
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